File: eagle_schematics/wag_chestpiece/wag_band/wagband_chestpiece_postroute.sch (EAGLE design)
At the start: 25 parts, among them U1 ATMEGA328P_PDIP, U2 TLV1117-33CDCY, U3 LM358DR, Y1 16MHz

Commit message: Fixed all schematics and boards to have separate power supplies finally :100:
Connections:
- removed net N$7: U$1.5/PWM, U$4.GPIO2
- removed net VCC: C1.1, C2.1, LED1.A, MPU6050_BREAKOUT.VCC, PWR.A, R2.2, R3.2, R5.2, U$1.VIN, U$2.3V3, U$4.CH_PD, U$4.TXD, U$5.P$1, U1.VCC, U2.INPUT, U2.OUTPUT, U3.VCC
- new net +3V3: C2.1, PWR.A, R5.2, U$2.3V3, U$4.RST, U$4.VCC, U1.VCC, U2.OUTPUT
- new net N$24: U$1.7/RX3, U$4.GPIO2
- new net V+: C1.1, LED1.A, MPU6050_BREAKOUT.VCC, R2.2, R3.2, U$1.VIN, U$5.P$1, U2.INPUT, U3.VCC
- net !RST: now also U$4.CH_PD; no longer U$4.RST
- net GND: now also U$4.GND; no longer U$4.RXD
- net N$19: now also U$4.TXD; no longer U$4.VCC
- net N$2: now also U$4.RXD; no longer U$4.GND
Other:
- moved on the sheet: U$4
