File: eagle_schematics/wag_chestpiece/wag_band/wagband_chestpiece_pre_route.brd (EAGLE design)
At the start: 66 x 66 mm, 25 parts, among them U1 ATMEGA328P_PDIP, U2 TLV1117-33CDCY, U3 LM358DR, Y1 16MHz

Commit message: Fixed all schematics and boards to have separate power supplies finally :100:
Connections:
- removed net N$7: U$1.5, U$4.GPIO2
- removed net VCC: C1.1, C2.1, LED1.A, MPU6050_BREAKOUT.VCC, PWR.A, R2.2, R3.2, R5.2, U$1.VIN, U$2.P$13, U$4.CH_PD, U$4.TX, U$5.P$1, U1.7, U2.3, U2.4, U3.8
- new net +3V3: C2.1, PWR.A, R5.2, U$2.P$13, U$4.RST, U$4.VCC, U1.7, U2.4
- new net N$24: U$1.7, U$4.GPIO2
- new net V+: C1.1, LED1.A, MPU6050_BREAKOUT.VCC, R2.2, R3.2, U$1.VIN, U$5.P$1, U2.3, U3.8
- net !RST: now also U$4.CH_PD; no longer U$4.RST
- net GND: now also U$4.GND; no longer U$4.RX
- net N$19: now also U$4.TX; no longer U$4.VCC
- net N$2: now also U$4.RX; no longer U$4.GND
Routing:
- removed copper zone on layer 1, net GND
- removed copper zone on layer 16, net GND
